Commit message: Add files via upload

File: car_4ws_4wd/urdf/car_4ws_4wd_gazebo.urdf (robot description, URDF)
Before this commit: robot car_4ws_4wd, 11 links, 10 joints
Links:
- link fl_drive_link: geometry collision mesh filename=package://car_4ws_4wd/meshes/fl_drive_link.STL; visual mesh filename=package://car_4ws_4wd/meshes/fl_drive_link.STL
- link fr_drive_link: geometry collision mesh filename=package://car_4ws_4wd/meshes/fr_drive_link.STL; visual mesh filename=package://car_4ws_4wd/meshes/fr_drive_link.STL
- link rl_drive_link: geometry collision mesh filename=package://car_4ws_4wd/meshes/rl_drive_link.STL; visual mesh filename=package://car_4ws_4wd/meshes/rl_drive_link.STL
- link rr_drive_link: geometry collision mesh filename=package://car_4ws_4wd/meshes/rr_drive_link.STL; visual mesh filename=package://car_4ws_4wd/meshes/rr_drive_link.STL
