Commit message: Add files via upload
添加雷达

File: car_4ws_4wd/urdf/car_4ws_4wd.urdf (robot description, URDF)
Before this commit: robot car_4ws_4wd, 10 links, 9 joints
Links:
- removed link base
- added link lidar_link, mass 0.3927; collision mesh filename=package://car_4ws_4wd/meshes/lidar_link.STL; visual mesh filename=package://car_4ws_4wd/meshes/lidar_link.STL
- link base_link: mass 40.395 -> 40.2533565247656
- link fl_drive_link: mass 2.1666 -> 2.16662276325971
- link fr_drive_link: mass 2.1666 -> 2.16662276325971
- link rl_drive_link: mass 2.1666 -> 2.16662276325971
Joints:
- removed joint base_joint
- added joint lidar_joint: type fixed, parent base_link, child lidar_link, origin xyz=0 0 0.565 rpy=0 0 0, axis 0 0 0
- joint fl_drive_joint: axis 0 0 -1 -> 0 0 1; origin xyz=0 0 -0.16 rpy=1.5708 0 0 -> xyz=0 0 -0.16 rpy=1.5707963267949 0 0
- joint fl_steer_joint: axis 0 0 1 -> 0 0 -1
- joint fr_drive_joint: axis 0 0 -1 -> 0 0 1; origin xyz=0 0 -0.16 rpy=1.5708 0 0 -> xyz=0 0 -0.16 rpy=1.5707963267949 0 0
- joint fr_steer_joint: axis 0 0 1 -> 0 0 -1; origin xyz=0.32 -0.235 -0.01 rpy=0 0 0 -> xyz=0.32 -0.235 -0.00999999999999999 rpy=0 0 0
- joint rl_drive_joint: axis 0 0 -1 -> 0 0 1; origin xyz=0 0 -0.16 rpy=1.5708 0 0 -> xyz=0 0 -0.16 rpy=1.5707963267949 0 0
- joint rl_steer_joint: axis 0 0 1 -> 0 0 -1
- joint rr_drive_joint: axis 0 0 -1 -> 0 0 1; origin xyz=0 0 -0.16 rpy=1.5708 0 0 -> xyz=0 0 -0.16 rpy=1.5707963267949 0 0
- joint rr_steer_joint: axis 0 0 1 -> 0 0 -1

File: car_4ws_4wd/urdf/car_4ws_4wd_gazebo.urdf (robot description, URDF)
Before this commit: robot car_4ws_4wd, 10 links, 9 joints
Links:
- added link lidar_link, mass 0.3927; collision mesh filename=package://car_4ws_4wd/meshes/lidar_link.STL; visual mesh filename=package://car_4ws_4wd/meshes/lidar_link.STL
- link base_link: mass 40.395 -> 40.2533565247656
- link fl_drive_link: mass 2.1666 -> 2.16662276325971; geometry collision cylinder length=0.05 radius=0.13; visual mesh filename=package://car_4ws_4wd/meshes/fl_drive_link.STL
- link fr_drive_link: mass 2.1666 -> 2.16662276325971; geometry collision cylinder length=0.05 radius=0.13; visual mesh filename=package://car_4ws_4wd/meshes/fr_drive_link.STL
- link rl_drive_link: mass 2.1666 -> 2.16662276325971; geometry collision cylinder length=0.05 radius=0.13; visual mesh filename=package://car_4ws_4wd/meshes/rl_drive_link.STL
- link rr_drive_link: geometry collision cylinder length=0.05 radius=0.13; visual mesh filename=package://car_4ws_4wd/meshes/rr_drive_link.STL
Joints:
- added joint lidar_joint: type fixed, parent base_link, child lidar_link, origin xyz=0 0 0.565 rpy=0 0 0, axis 0 0 0
- joint fl_drive_joint: origin xyz=0 0 -0.16 rpy=1.5708 0 0 -> xyz=0 0 -0.16 rpy=1.5707963267949 0 0
- joint fr_drive_joint: origin xyz=0 0 -0.16 rpy=1.5708 0 0 -> xyz=0 0 -0.16 rpy=1.5707963267949 0 0
- joint fr_steer_joint: origin xyz=0.32 -0.235 -0.01 rpy=0 0 0 -> xyz=0.32 -0.235 -0.00999999999999999 rpy=0 0 0
- joint rl_drive_joint: origin xyz=0 0 -0.16 rpy=1.5708 0 0 -> xyz=0 0 -0.16 rpy=1.5707963267949 0 0
- joint rr_drive_joint: origin xyz=0 0 -0.16 rpy=1.5708 0 0 -> xyz=0 0 -0.16 rpy=1.5707963267949 0 0

Commit message: Add files via upload

File: car_4ws_4wd/urdf/car_4ws_4wd.urdf (robot description, URDF)
Before this commit: robot car_4ws_4wd, 10 links, 9 joints
Joints:
- joint fl_drive_joint: axis 0 0 1 -> 0 0 -1
- joint fl_steer_joint: axis 0 0 -1 -> 0 0 1
- joint fr_drive_joint: axis 0 0 1 -> 0 0 -1
- joint fr_steer_joint: axis 0 0 -1 -> 0 0 1
- joint rl_drive_joint: axis 0 0 1 -> 0 0 -1
- joint rl_steer_joint: axis 0 0 -1 -> 0 0 1
- joint rr_drive_joint: axis 0 0 1 -> 0 0 -1
- joint rr_steer_joint: axis 0 0 -1 -> 0 0 1

Commit message: Add files via upload

File: car_4ws_4wd/urdf/car_4ws_4wd.urdf (robot description, URDF)
Before this commit: robot car_4ws_4wd, 10 links, 9 joints
Links:
- link fl_drive_link: geometry collision cylinder length=0.05 radius=0.13; visual mesh filename=package://car_4ws_4wd/meshes/fl_drive_link.STL
- link fr_drive_link: geometry collision cylinder length=0.05 radius=0.13; visual mesh filename=package://car_4ws_4wd/meshes/fr_drive_link.STL
- link rl_drive_link: geometry collision cylinder length=0.05 radius=0.13; visual mesh filename=package://car_4ws_4wd/meshes/rl_drive_link.STL
- link rr_drive_link: geometry collision cylinder length=0.05 radius=0.13; visual mesh filename=package://car_4ws_4wd/meshes/rr_drive_link.STL
Joints:
- joint fl_drive_joint: axis 0 0 -1 -> 0 0 1
- joint fl_steer_joint: axis 0 0 1 -> 0 0 -1; limit lower=-0.55 upper=0.55 effort=100 velocity=1 -> lower=-0.55 upper=0.55 effort=50 velocity=1
- joint fr_drive_joint: axis 0 0 -1 -> 0 0 1
- joint fr_steer_joint: axis 0 0 1 -> 0 0 -1; limit lower=-0.55 upper=0.55 effort=100 velocity=1 -> lower=-0.55 upper=0.55 effort=50 velocity=1
- joint rl_drive_joint: axis 0 0 -1 -> 0 0 1
- joint rl_steer_joint: axis 0 0 1 -> 0 0 -1; limit lower=-0.55 upper=0.55 effort=100 velocity=1 -> lower=-0.55 upper=0.55 effort=50 velocity=1
- joint rr_drive_joint: axis 0 0 -1 -> 0 0 1
- joint rr_steer_joint: axis 0 0 1 -> 0 0 -1; limit lower=-0.55 upper=0.55 effort=100 velocity=1 -> lower=-0.55 upper=0.55 effort=50 velocity=1

File: car_4ws_4wd/urdf/car_4ws_4wd.urdf.xacro (robot description, xacro)
@@ -81,5 +81,5 @@
         <origin xyz="0 0 0" rpy="0 0 0" />
         <geometry>
-          <mesh filename="${mesh_path}/${prefix}_drive_link.STL" />
+          <cylinder radius="0.13" length="0.05"/>
         </geometry>
       </collision>

File: car_4ws_4wd/urdf/car_4ws_4wd_gazebo.urdf (robot description, URDF)
Before this commit: robot car_4ws_4wd, 11 links, 10 joints
Links:
- link fl_drive_link: geometry collision cylinder length=0.05 radius=0.13; visual mesh filename=package://car_4ws_4wd/meshes/fl_drive_link.STL
- link fr_drive_link: geometry collision cylinder length=0.05 radius=0.13; visual mesh filename=package://car_4ws_4wd/meshes/fr_drive_link.STL
- link rl_drive_link: geometry collision cylinder length=0.05 radius=0.13; visual mesh filename=package://car_4ws_4wd/meshes/rl_drive_link.STL
- link rr_drive_link: geometry collision cylinder length=0.05 radius=0.13; visual mesh filename=package://car_4ws_4wd/meshes/rr_drive_link.STL
